Commit message: made copies of repo files to be replaced for ones installed with apt

File: kortex_description/grippers/robotiq_2f_85/urdf/robotiq_2f_85_macro_repo.xacro (robot description, xacro)
@@ -8,5 +8,7 @@
     sim_ignition:=false
     sim_isaac:=false
-    use_internal_bus_gripper_comm:=true">
+    isaac_joint_commands:=/isaac_joint_commands
+    isaac_joint_states:=/isaac_joint_states
+    use_internal_bus_gripper_comm:=false">
     <xacro:include filename="$(find robotiq_description)/urdf/robotiq_2f_85_macro.urdf.xacro" />
     <!-- Hardware talks directly to the gripper so we don't need ros2_control unless we are simulating -->
@@ -20,8 +22,10 @@
         parent="${parent}"
         include_ros2_control="${include_ros2_control}"
-        use_fake_hardware="$(arg use_fake_hardware)"
-        fake_sensor_commands="$(arg fake_sensor_commands)"
-        sim_ignition="$(arg sim_ignition)"
-        sim_isaac="$(arg sim_isaac)">
+        use_fake_hardware="${use_fake_hardware}"
+        fake_sensor_commands="${fake_sensor_commands}"
+        sim_ignition="${sim_ignition}"
+        sim_isaac="${sim_isaac}"
+        isaac_joint_commands="${isaac_joint_commands}"
+        isaac_joint_states="${isaac_joint_states}">
         <origin xyz="0 0 0" rpy="0 0 0" />
     </xacro:robotiq_gripper>

File: kortex_description/robots/gen3_repo.xacro (robot description, xacro)
@@ -25,4 +25,8 @@
     <xacro:arg name="use_external_cable" default="false" />
     <xacro:include filename="$(find kortex_description)/robots/kortex_robot.xacro" />
+    <!-- initial position for simulations (Mock Hardware, Gazebo, Ignition) -->
+    <xacro:arg name="initial_positions_file" default="$(find kortex_description)/config/initial_positions.yaml"/>
+    <!-- convert to property to use substitution in function -->
+    <xacro:property name="initial_positions_file" default="$(arg initial_positions_file)"/>
     <link name="world" />
     <xacro:load_robot
@@ -49,5 +53,6 @@
         sim_ignition="$(arg sim_ignition)"
         sim_isaac="$(arg sim_isaac)"
-        use_external_cable="$(arg use_external_cable)" >
+        use_external_cable="$(arg use_external_cable)"
+        initial_positions="${xacro.load_yaml(initial_positions_file)}" >
         <origin xyz="0 0 0" rpy="0 0 0" />  <!-- position robot in the world -->
     </xacro:load_robot>

File: kortex_description/robots/kortex_robot_repo.xacro (robot description, xacro)
@@ -23,5 +23,8 @@
     sim_ignition:=false
     sim_isaac:=false
+    isaac_joint_commands:=/isaac_joint_commands
+    isaac_joint_states:=/isaac_joint_states
     use_external_cable:=false
+    initial_positions:=${dict(joint_1=0.0,joint_2=0.0,joint_3=0.0,joint_4=0.0,joint_5=0.0,joint_6=0.0,joint_7=0.0)}
     gripper_max_velocity:=100.0
     gripper_max_force:=100.0">
@@ -47,8 +50,11 @@
       sim_ignition="${sim_ignition}"
       sim_isaac="${sim_isaac}"
+      isaac_joint_commands="${isaac_joint_commands}"
+      isaac_joint_states="${isaac_joint_states}"
       gripper_joint_name="${gripper_joint_name}"
       gripper_max_velocity="${gripper_max_velocity}"
       gripper_max_force="${gripper_max_force}"
-      use_external_cable="${use_external_cable}">
+      use_external_cable="${use_external_cable}"
+      initial_positions="${initial_positions}">
       <xacro:insert_block name="origin" />
     </xacro:load_arm>
@@ -73,5 +79,8 @@
         fake_sensor_commands="${fake_sensor_commands}"
         sim_ignition="${sim_ignition}"
-        sim_isaac="${sim_isaac}"/>
+        sim_isaac="${sim_isaac}"
+        isaac_joint_commands="${isaac_joint_commands}"
+        isaac_joint_states="${isaac_joint_states}"
+        use_internal_bus_gripper_comm="${use_internal_bus_gripper_comm}"/>
     </xacro:unless>
   </xacro:macro>
